File: pcb/BERTV3.kicad_sch (KiCad schematic)
At the start: 3 parts

Commit message: first draft schematic
Parts:
- added BT?: Battery, symbol Device:Battery
- added C? (x2): C, symbol Device:C
- added SW?: SW_SPST, symbol Switch:SW_SPST
- added U?: INA219-BOB, symbol HAR:INA219-BOB
- added U?: AZ1117-3.3, symbol Regulator_Linear:AZ1117-3.3
Connections:
- net at U?.1 (EXT_SW+): now also SW?.1 (A)
- net at U?.2 (EXT_SW-): now also SW?.2 (B)
- net at U?.6 (5VOUT+): now also C?.1, U?.1 (V+)
- net GND: now reaches U?.7 (5VOUT-)
- net GND: now also U?.1 (GND), U?.2 (GND), U?.9 (BATT-), BT?.2 (-), C?.2, C?.2, U?.1 (GND)
- net at U?.8 (BATT+): now also BT?.1 (+)
- net at U?.3 (3V3): now also C?.1, U?.2 (VO)
- new net: U?.2 (V-), U?.3 (VI)
- no-connect marks 0 -> 19
Other:
- moved on the sheet: U?
